Commit message: Add the base link

File: description/robot.urdf.xacro (robot description, xacro)
@@ -4,5 +4,5 @@
   <xacro:include filename="colors.xacro" />
   <xacro:include filename="gazebo_control.xacro" />
-  <!-- Base Link-->
+  <!-- Base Link -->
   <link name="base_link">
   </link>
@@ -44,4 +44,11 @@
     </collision>
   </link>
+  <joint
+  name="rear_chassis_joint"
+  type="fixed">
+    <parent link="base_link" />
+    <child link="rear_chassis" />
+    <origin xyz="0.625 0 0.790" />
+  </joint>
   <gazebo reference="rear_chassis">
 		<material>Gazebo/green</material>
